File: FAP_modules/io_board/io_board.sch (EAGLE design)
At the start: 74 parts, among them IC1 STM32F051C8T6, IC2 EPM240-T100, IC3 24C08BSN, U2 OSCILLATORSMD

Commit message: WAIT and interrupt chaining on IO board
Parts:
- added JP5, JP6: (no value), pinhead:PINHD-1X1
- added LED10, LED11: (no value), adafruit:LEDCHIP-LED0805
- added R26, R27: (no value), SparkFun-Passives:RESISTOR0805-RES
- LED1, LED3, LED4, LED5, LED6, LED7, LED8, LED9: device adafruit:LEDCHIPLED_0805 -> adafruit:LEDCHIP-LED0805
- U$1: value FAP_BUS -> FAP_BUS_FAP_BUS; device vga_pcb:FAP_BUS -> cpu_board:FAP_BUS_FAP_BUS
Connections:
- new net N$100: IC2B1.IOB1-41, U$1.30
- new net N$101: IC2B1.IOB1-40, U$1.40
- new net N$102: LED10.A, R26.2
- new net N$103: IC2B1.IOB1-16, JP5.1, LED10.C
- new net N$104: LED11.A, R27.2
- new net N$105: IC2B1.IOB1-19, JP6.1, LED11.C
- new net N$99: IC2B2.IOB2-69, U$1.29
- net +3V3: now also R26.1, R27.1, R6.1
- net GND: no longer R6.1
- net N$23: now also U$1.39; no longer U$1.29
- net N$73: now also LED1.C; no longer IC2B1.IOB1-16, LED1.A
- net N$74: now also LED1.A; no longer LED1.C
Other:
- moved on the sheet: LED1
