File: FAP_modules/io_board/io_board.brd (EAGLE design)
At the start: 100 x 60 mm, 84 parts, among them IC1 STM32F051C8T6, IC2 EPM240-T100, IC3 24C08BSN, U2 OSCILLATORSMD

Commit message: board cleanup
Routing:
- net TCK: track 58.4 -> 57.0 mm
Changed lines of the file:
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@@
 <via x="49.403" y="25.908" extent="1-16" drill="0.5"/>
 <wire x1="49.403" y1="25.908" x2="50.927" y2="24.384" width="0.254" layer="16"/>
-<wire x1="50.927" y1="24.384" x2="54.229" y2="24.384" width="0.254" layer="16"/>
-<wire x1="54.229" y1="24.384" x2="55.626" y2="22.987" width="0.254" layer="16"/>
-<wire x1="55.626" y1="22.987" x2="90.297" y2="22.987" width="0.254" layer="16"/>
-<wire x1="90.297" y1="22.987" x2="91.821" y2="21.463" width="0.254" layer="16"/>
-<wire x1="91.821" y1="21.463" x2="93.599" y2="21.463" width="0.254" layer="16"/>
-<wire x1="93.599" y1="21.463" x2="95.25" y2="23.114" width="0.254" layer="16"/>
 <wire x1="95.134" y1="16.8656" x2="95.25" y2="16.9816" width="0.254" layer="1"/>
 <wire x1="95.25" y1="16.9816" x2="95.25" y2="23.114" width="0.254" layer="1"/>
+<wire x1="50.927" y1="24.384" x2="93.98" y2="24.384" width="0.254" layer="16"/>
+<wire x1="93.98" y1="24.384" x2="95.25" y2="23.114" width="0.254" layer="16"/>
 </signal>
 <signal name="TMS">
@@
 <wire x1="53.68518125" y1="14.785028125" x2="52.900009375" y2="15.5702" width="0.2032" layer="1"/>
 <wire x1="52.900009375" y1="15.5702" x2="51.308" y2="15.5702" width="0.2032" layer="1"/>
-<wire x1="43.686" y1="2.032" x2="41.146" y2="2.032" width="0" layer="19" extent="1-1"/>
 </signal>
 <signal name="+3V3">
@@
 <wire x1="51.181" y1="29.464" x2="51.181" y2="26.162" width="0.254" layer="16"/>
 <wire x1="51.181" y1="26.162" x2="52.324" y2="25.019" width="0.254" layer="16"/>
-<wire x1="52.324" y1="25.019" x2="59.944" y2="25.019" width="0.254" layer="16"/>
-<wire x1="59.944" y1="25.019" x2="60.452" y2="24.511" width="0.254" layer="16"/>
-<wire x1="60.452" y1="24.511" x2="88.392" y2="24.511" width="0.254" layer="16"/>
 <wire x1="90.805" y1="26.924" x2="93.98" y2="26.924" width="0.254" layer="16"/>
 <wire x1="93.98" y1="26.924" x2="95.25" y2="25.654" width="0.254" layer="16"/>
-<wire x1="88.392" y1="24.511" x2="90.805" y2="26.924" width="0.254" layer="16"/>
+<wire x1="52.324" y1="25.019" x2="88.9" y2="25.019" width="0.254" layer="16"/>
+<wire x1="88.9" y1="25.019" x2="90.805" y2="26.924" width="0.254" layer="16"/>
 </signal>
 <signal name="N$99">
@@
 <wire x1="48.006" y1="3.302" x2="47.498" y2="3.81" width="0.254" layer="16"/>
 <wire x1="47.498" y1="3.81" x2="47.498" y2="11.684" width="0.254" layer="16"/>
-<wire x1="47.498" y1="11.684" x2="45.974" y2="13.208" width="0.254" layer="16"/>
-<via x="45.974" y="13.208" extent="1-16" drill="0.5"/>
-<wire x1="45.974" y1="13.208" x2="45.390640625" y2="13.208" width="0.254" layer="1"/>
+<via x="46.7614" y="12.4968" extent="1-16" drill="0.5"/>
 <wire x1="45.390640625" y1="13.208" x2="44.139240625" y2="11.9566" width="0.254" layer="1"/>
+<wire x1="45.390640625" y1="13.208" x2="46.0502" y2="13.208" width="0.254" layer="1"/>
+<wire x1="46.0502" y1="13.208" x2="46.7614" y2="12.4968" width="0.254" layer="1"/>
+<wire x1="46.7614" y1="12.4968" x2="46.7614" y2="12.4206" width="0.254" layer="16"/>
+<wire x1="46.7614" y1="12.4206" x2="47.498" y2="11.684" width="0.254" layer="16"/>
 </signal>
 <signal name="N$100">
@@
 <wire x1="52.2732" y1="29.2862" x2="52.6796" y2="29.2862" width="0.2032" layer="16"/>
 <wire x1="52.6796" y1="29.2862" x2="53.34" y2="28.6258" width="0.2032" layer="16"/>
-<wire x1="53.34" y1="28.6258" x2="83.4898" y2="28.6258" width="0.2032" layer="16"/>
-<wire x1="83.4898" y1="28.6258" x2="86.5124" y2="25.6032" width="0.2032" layer="16"/>
-<via x="86.5124" y="25.6032" extent="1-16" drill="0.5"/>
-<wire x1="86.5124" y1="25.6032" x2="86.5124" y2="19.685" width="0.2032" layer="1"/>
+<wire x1="53.34" y1="28.6258" x2="84.0486" y2="28.6258" width="0.2032" layer="16"/>
+<via x="86.5124" y="26.162" extent="1-16" drill="0.5"/>
+<wire x1="86.5124" y1="26.162" x2="86.5124" y2="19.685" width="0.2032" layer="1"/>
 <wire x1="86.5124" y1="19.685" x2="99.2886" y2="6.9088" width="0.2032" layer="1"/>
 <wire x1="99.2886" y1="6.9088" x2="99.2886" y2="1.6256" width="0.2032" layer="1"/>
@@
 <wire x1="98.1456" y1="0.4826" x2="80.7954" y2="0.4826" width="0.2032" layer="1"/>
 <wire x1="80.7954" y1="0.4826" x2="79.246" y2="2.032" width="0.2032" layer="1"/>
+<wire x1="86.5124" y1="26.162" x2="84.0486" y2="28.6258" width="0.2032" layer="16"/>
 </signal>
 <signal name="N$4">

Commit message: board cleanup
Routing:
- net N$3: track 89.0 -> 88.3 mm
Other:
- board text added: "FAP80 I/O Board V2 dekuNukem 2016"
- board text removed: "FAP I/O Board V2 dekuNukem 2016"
Changed lines of the file:
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@@
 <wire x1="100" y1="60" x2="0" y2="60" width="0" layer="20"/>
 <wire x1="0" y1="60" x2="0" y2="0" width="0" layer="20"/>
-<text x="65.1764" y="19.304" size="1.6764" layer="25">FAP I/O Board V2
+<text x="65.1764" y="19.304" size="1.6764" layer="25">FAP80 I/O Board V2
 dekuNukem 2016</text>
 <circle x="3.7592" y="48.5902" radius="1.016" width="0" layer="41"/>
@@
 <via x="42.3418" y="43.5864" extent="1-16" drill="0.6"/>
 <via x="50.165" y="43.1546" extent="1-16" drill="0.5"/>
-<wire x1="53.79496875" y1="40.573009375" x2="52.5052875" y2="41.862690625" width="0.2032" layer="1"/>
 <wire x1="52.734309375" y1="39.512346875" x2="51.7906" y2="40.45605625" width="0.2032" layer="1"/>
 <wire x1="51.7906" y1="40.45605625" x2="51.7906" y2="41.021" width="0.2032" layer="1"/>
 <wire x1="51.7906" y1="41.021" x2="52.5052875" y2="41.7356875" width="0.2032" layer="1"/>
-<wire x1="52.5052875" y1="41.7356875" x2="52.5052875" y2="41.862690625" width="0.2032" layer="1"/>
 <contactref element="U$3" pad="GND"/>
 <contactref element="IC3" pad="4"/>
@@
 <wire x1="53.68518125" y1="14.785028125" x2="52.900009375" y2="15.5702" width="0.2032" layer="1"/>
 <wire x1="52.900009375" y1="15.5702" x2="51.308" y2="15.5702" width="0.2032" layer="1"/>
+<wire x1="53.79496875" y1="40.573009375" x2="52.632290625" y2="41.7356875" width="0.2032" layer="1"/>
+<wire x1="52.632290625" y1="41.7356875" x2="52.5052875" y2="41.7356875" width="0.2032" layer="1"/>
 </signal>
 <signal name="+3V3">
@@
 <wire x1="53.34" y1="28.6258" x2="84.0486" y2="28.6258" width="0.2032" layer="16"/>
 <via x="86.5124" y="26.162" extent="1-16" drill="0.5"/>
-<wire x1="86.5124" y1="26.162" x2="86.5124" y2="19.685" width="0.2032" layer="1"/>
-<wire x1="86.5124" y1="19.685" x2="99.2886" y2="6.9088" width="0.2032" layer="1"/>
-<wire x1="99.2886" y1="6.9088" x2="99.2886" y2="1.6256" width="0.2032" layer="1"/>
-<wire x1="99.2886" y1="1.6256" x2="98.1456" y2="0.4826" width="0.2032" layer="1"/>
-<wire x1="98.1456" y1="0.4826" x2="80.7954" y2="0.4826" width="0.2032" layer="1"/>
-<wire x1="80.7954" y1="0.4826" x2="79.246" y2="2.032" width="0.2032" layer="1"/>
+<wire x1="86.5124" y1="26.162" x2="86.5124" y2="19.2024" width="0.254" layer="1"/>
+<wire x1="98.7806" y1="6.9342" x2="98.7806" y2="1.3208" width="0.254" layer="1"/>
+<wire x1="98.171" y1="0.7112" x2="80.5668" y2="0.7112" width="0.254" layer="1"/>
 <wire x1="86.5124" y1="26.162" x2="84.0486" y2="28.6258" width="0.2032" layer="16"/>
+<wire x1="86.5124" y1="19.2024" x2="98.7806" y2="6.9342" width="0.254" layer="1"/>
+<wire x1="98.7806" y1="1.3208" x2="98.171" y2="0.7112" width="0.254" layer="1"/>
+<wire x1="80.5668" y1="0.7112" x2="79.246" y2="2.032" width="0.254" layer="1"/>
 </signal>
 <signal name="N$4">

Commit message: firmware updates
Parts:
- added R28: (no value), SparkFun-Passives:0805
- moved R3 2.87 mm to (26.9, 51.7)
Connections:
- new net N$108: R28.1, U$3.GPIO2
- net +3V3: now also R28.2, U$3.CH_PD
- net N$68: no longer U$3.CH_PD, U$3.GPIO2
Routing:
- net N$108: track 0.00 -> 6.02 mm
- net N$68: track 8.11 -> 6.35 mm
Changed lines of the file:
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@@
 <attribute name="VALUE" x="36.7538" y="54.2036" size="0.4064" layer="27" rot="R90"/>
 </element>
-<element name="R3" library="SparkFun-Passives" package="0805" value="" x="24.0792" y="51.308" smashed="yes">
-<attribute name="NAME" x="26.289" y="50.9397" size="0.8128" layer="25"/>
-<attribute name="VALUE" x="23.0632" y="49.911" size="0.4064" layer="27"/>
+<element name="R3" library="SparkFun-Passives" package="0805" value="" x="26.924" y="51.689" smashed="yes">
+<attribute name="NAME" x="26.4668" y="49.6189" size="0.8128" layer="25"/>
+<attribute name="VALUE" x="25.908" y="50.292" size="0.4064" layer="27"/>
 </element>
 <element name="SD1" library="Adafruit Feather M0 Adalogger" package="TF-PULL" value="TF-HOLDER" x="7.0104" y="43.688" smashed="yes" rot="R90"/>
@@
 <element name="TP9" library="SparkFun-Passives" package="PAD.03X.04" value="TEST-POINT3X4" x="56.3626" y="12.8524"/>
 <element name="TP10" library="SparkFun-Passives" package="PAD.03X.04" value="TEST-POINT3X4" x="56.1594" y="14.478"/>
+<element name="R28" library="SparkFun-Passives" package="0805" value="" x="23.495" y="51.689" smashed="yes">
+<attribute name="NAME" x="22.8092" y="49.6951" size="0.8128" layer="25"/>
+<attribute name="VALUE" x="22.479" y="50.292" size="0.4064" layer="27"/>
+</element>
 </elements>
 <signals>
@@
 <wire x1="38.2016" y1="23.4696" x2="36.85679375" y2="24.81440625" width="0.2032" layer="1"/>
 <wire x1="36.85679375" y1="24.81440625" x2="36.85679375" y2="25.373203125" width="0.2032" layer="1"/>
+<contactref element="U$3" pad="CH_PD"/>
+<contactref element="R28" pad="2"/>
 <wire x1="36.85679375" y1="25.373203125" x2="36.9316" y2="25.3238" width="0" layer="19" extent="1-1"/>
 <wire x1="40.60370625" y1="15.492134375" x2="42.017921875" y2="14.077921875" width="0" layer="19" extent="1-1"/>
@@
 <signal name="N$68">
 <contactref element="R3" pad="1"/>
-<contactref element="U$3" pad="GPIO2"/>
 <contactref element="U$3" pad="GPIO0"/>
-<contactref element="U$3" pad="CH_PD"/>
-<wire x1="23.1752" y1="56.8719" x2="25.7152" y2="56.8719" width="0.254" layer="16"/>
-<wire x1="23.1752" y1="56.8719" x2="23.1752" y2="54.3319" width="0.254" layer="16"/>
-<wire x1="23.1752" y1="54.3319" x2="23.1792" y2="54.3279" width="0.254" layer="1"/>
-<wire x1="23.1792" y1="54.3279" x2="23.1792" y2="51.308" width="0.254" layer="1"/>
+<wire x1="26.024" y1="51.689" x2="24.4602" y2="53.2528" width="0.254" layer="1"/>
+<wire x1="24.4602" y1="53.2528" x2="24.4602" y2="55.3974" width="0.254" layer="1"/>
+<wire x1="24.4602" y1="55.3974" x2="25.7152" y2="56.6524" width="0.254" layer="1"/>
+<wire x1="25.7152" y1="56.6524" x2="25.7152" y2="56.8719" width="0.254" layer="1"/>
 </signal>
 <signal name="N$69">
@@
 <wire x1="55.406425" y1="14.478" x2="56.1594" y2="14.478" width="0.254" layer="1"/>
 </signal>
+<signal name="N$108">
+<contactref element="U$3" pad="GPIO2"/>
+<contactref element="R28" pad="1"/>
+<wire x1="22.595" y1="51.689" x2="21.8694" y2="52.4146" width="0.254" layer="1"/>
+<wire x1="21.8694" y1="52.4146" x2="21.8694" y2="55.1688" width="0.254" layer="1"/>
+<wire x1="21.8694" y1="55.1688" x2="23.1752" y2="56.4746" width="0.254" layer="1"/>
+<wire x1="23.1752" y1="56.4746" x2="23.1752" y2="56.8719" width="0.254" layer="1"/>
+</signal>
 </signals>
