File: FAP_modules/backplane/backplane.sch (EAGLE design)
At the start: 45 parts, among them IC1 REG1117, J1 USB-MICROB, U1 STM32F10XRXT6

Commit message: added GND test headers
Parts:
- added JP5: (no value), pinhead:PINHD-1X2
- R2: value 10K -> 1K5
Connections:
- net GND: now also JP5.1, JP5.2
Changed lines of the file:
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@@
 <?xml version="1.0" encoding="utf-8"?>
 <!DOCTYPE eagle SYSTEM "eagle.dtd">
-<eagle version="7.6.0">
+<eagle version="7.7.0">
 <drawing>
 <settings>
@@
 <part name="GND17" library="supply1" deviceset="GND" device=""/>
 <part name="GND18" library="supply1" deviceset="GND" device=""/>
-<part name="R2" library="SparkFun-Passives" deviceset="RESISTOR" device="0805-RES" value="10K"/>
+<part name="R2" library="SparkFun-Passives" deviceset="RESISTOR" device="0805-RES" value="1K5"/>
 <part name="C12" library="SparkFun-Capacitors" deviceset="CAP" device="0805" value="100nF"/>
 <part name="GND22" library="supply1" deviceset="GND" device=""/>
@@
 <part name="U$13" library="m3_mounting_hole" deviceset="M3_MOUNTING_HOLE" device=""/>
 <part name="U$14" library="m3_mounting_hole" deviceset="M3_MOUNTING_HOLE" device=""/>
+<part name="JP5" library="pinhead" deviceset="PINHD-1X2" device=""/>
+<part name="GND3" library="supply1" deviceset="GND" device=""/>
 </parts>
 <sheets>
@@
 </instance>
 <instance part="GND9" gate="1" x="495.3" y="-60.96"/>
-<instance part="U$3" gate="G$1" x="287.02" y="-91.44"/>
+<instance part="U$3" gate="G$1" x="231.14" y="-68.58"/>
 <instance part="GND10" gate="1" x="307.34" y="35.56"/>
 <instance part="P+6" gate="1" x="322.58" y="152.4" rot="MR0"/>
@@
 <attribute name="VALUE" x="-3.556" y="61.341" size="1.778" layer="96"/>
 </instance>
-<instance part="GND22" gate="1" x="5.08" y="50.8"/>
-<instance part="+3V8" gate="G$1" x="7.62" y="76.2"/>
+<instance part="GND22" gate="1" x="2.54" y="50.8"/>
+<instance part="+3V8" gate="G$1" x="2.54" y="76.2"/>
 <instance part="U$4" gate="G$1" x="335.28" y="109.22"/>
 <instance part="U$1" gate="G$1" x="518.16" y="109.22"/>
@@
 <instance part="+3V2" gate="G$1" x="-109.22" y="73.66"/>
 <instance part="U$7" gate="G$1" x="-50.8" y="-25.4"/>
-<instance part="U$8" gate="G$1" x="-53.34" y="-40.64"/>
-<instance part="U$9" gate="G$1" x="-55.88" y="-55.88"/>
-<instance part="U$10" gate="G$1" x="-55.88" y="-73.66"/>
-<instance part="U$11" gate="G$1" x="22.86" y="-43.18"/>
-<instance part="U$12" gate="G$1" x="22.86" y="-60.96"/>
-<instance part="U$13" gate="G$1" x="25.4" y="-76.2"/>
-<instance part="U$14" gate="G$1" x="25.4" y="-96.52"/>
+<instance part="U$8" gate="G$1" x="-50.8" y="-40.64"/>
+<instance part="U$9" gate="G$1" x="-50.8" y="-55.88"/>
+<instance part="U$10" gate="G$1" x="-50.8" y="-73.66"/>
+<instance part="U$11" gate="G$1" x="-15.24" y="-25.4"/>
+<instance part="U$12" gate="G$1" x="-15.24" y="-40.64"/>
+<instance part="U$13" gate="G$1" x="-15.24" y="-55.88"/>
+<instance part="U$14" gate="G$1" x="-15.24" y="-73.66"/>
+<instance part="JP5" gate="G$1" x="566.42" y="7.62"/>
+<instance part="GND3" gate="1" x="553.72" y="5.08"/>
 </instances>
 <busses>
@@
 <pinref part="C12" gate="G$1" pin="2"/>
 <wire x1="2.54" y1="60.96" x2="2.54" y2="53.34" width="0.1524" layer="91"/>
-<wire x1="2.54" y1="53.34" x2="5.08" y2="53.34" width="0.1524" layer="91"/>
 <pinref part="GND22" gate="1" pin="GND"/>
 </segment>
@@
 <junction x="-124.46" y="63.5"/>
 <pinref part="GND1" gate="1" pin="GND"/>
+</segment>
+<segment>
+<pinref part="JP5" gate="G$1" pin="1"/>
+<pinref part="GND3" gate="1" pin="GND"/>
+<wire x1="563.88" y1="10.16" x2="553.72" y2="10.16" width="0.1524" layer="91"/>
+<wire x1="553.72" y1="10.16" x2="553.72" y2="7.62" width="0.1524" layer="91"/>
+<pinref part="JP5" gate="G$1" pin="2"/>
+<wire x1="563.88" y1="7.62" x2="553.72" y2="7.62" width="0.1524" layer="91"/>
+<junction x="553.72" y="7.62"/>
 </segment>
 </net>
@@
 <pinref part="C12" gate="G$1" pin="1"/>
 <wire x1="2.54" y1="68.58" x2="2.54" y2="73.66" width="0.1524" layer="91"/>
-<wire x1="2.54" y1="73.66" x2="7.62" y2="73.66" width="0.1524" layer="91"/>
 <pinref part="+3V8" gate="G$1" pin="+3V3"/>
 </segment>

Commit message: added interrupt chaining and WAIT
Parts:
- removed JP5: (no value), pinhead:PINHD-1X2
- removed R2: 1K5, SparkFun-Passives:RESISTOR0805-RES
- added JP2: (no value), adafruit:PINHD-1X1
- added LED1: (no value), adafruit:LEDCHIP-LED0805
- added R1: (no value), adafruit:R-US_R0805
- J1: device SparkFun-Connectors:USB-MICROB -> v3:USB-MICROB
Connections:
- removed net N$19: JP3.29, U$1.29, U$2.29, U$4.29, U$5.29, U$6.29, U1PORTC_L.PC3
- new net N$1: JP3.29, U$6.29
- new net N$10: U$2.29, U$5.39
- new net N$12: LED1.C, R1.2
- new net N$15: JP3.WAIT, U$1.WAIT, U$2.WAIT, U$4.WAIT, U$5.WAIT, U$6.WAIT
- new net N$2: U$5.29, U$6.39
- new net N$5: U$1.39, U$4.29
- new net N$6: U$1.29, U$2.39
- new net N$8: U$4.39, U1PORTC_L.PC3
- net GND: now also JP3.GND, R1.1; no longer JP5.1, JP5.2
- net N$61: now also JP2.1, LED1.A; no longer R2.1
- net N$96: no longer R2.2

Commit message: added all Z80 signals on bus
Parts:
- removed JP2: (no value), adafruit:PINHD-1X1
Connections:
- removed net N$15: JP3.WAIT, U$1.WAIT, U$2.WAIT, U$4.WAIT, U$5.WAIT, U$6.WAIT
- removed net N$61: JP2.1, LED1.A, U1PORTA_H.PA10
- new net N$19: JP3.REFRESH, U$1.REFRESH, U$2.REFRESH, U$4.REFRESH, U$5.REFRESH, U$6.REFRESH
- new net N$21: JP3.HALT, U$1.HALT, U$2.HALT, U$4.HALT, U$5.HALT, U$6.HALT, U1PORTC_H.PC9
- new net N$27: JP3.WAIT, U$1.WAIT, U$2.WAIT, U$4.WAIT, U$5.WAIT, U$6.WAIT, U1PORTA_H.PA10
- net +3V3: now also LED1.A
- net GND: no longer R1.1
- net N$67: now also R1.1
Other:
- moved on the sheet: LED1, R1
Changed lines of the file:
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@@
 <part name="LED1" library="adafruit" deviceset="LED" device="CHIP-LED0805"/>
 <part name="R1" library="adafruit" deviceset="R-US_" device="R0805"/>
-<part name="GND2" library="supply1" deviceset="GND" device=""/>
-<part name="JP2" library="adafruit" deviceset="PINHD-1X1" device=""/>
 <part name="GND4" library="supply1" deviceset="GND" device=""/>
+<part name="+3V3" library="supply1" deviceset="+3V3" device=""/>
 </parts>
 <sheets>
@@
 <instance part="U$13" gate="G$1" x="-15.24" y="-55.88"/>
 <instance part="U$14" gate="G$1" x="-15.24" y="-73.66"/>
-<instance part="LED1" gate="G$1" x="144.78" y="106.68"/>
-<instance part="R1" gate="G$1" x="144.78" y="96.52" rot="R90"/>
-<instance part="GND2" gate="1" x="144.78" y="88.9"/>
-<instance part="JP2" gate="G$1" x="162.56" y="99.06"/>
+<instance part="LED1" gate="G$1" x="238.76" y="137.16"/>
+<instance part="R1" gate="G$1" x="238.76" y="127" rot="R90"/>
 <instance part="GND4" gate="1" x="662.94" y="38.1"/>
+<instance part="+3V3" gate="G$1" x="238.76" y="142.24"/>
 </instances>
 <busses>
@@
 </segment>
 <segment>
-<pinref part="R1" gate="G$1" pin="1"/>
-<pinref part="GND2" gate="1" pin="GND"/>
-</segment>
-<segment>
 <pinref part="JP3" gate="-1" pin="GND"/>
 <pinref part="GND4" gate="1" pin="GND"/>
@@
 <pinref part="+3V2" gate="G$1" pin="+3V3"/>
 </segment>
+<segment>
+<pinref part="LED1" gate="G$1" pin="A"/>
+<pinref part="+3V3" gate="G$1" pin="+3V3"/>
+</segment>
 </net>
 <net name="N$14" class="0">
@@
 </segment>
 </net>
-<net name="N$61" class="0">
-<segment>
-<wire x1="144.78" y1="109.22" x2="152.4" y2="109.22" width="0.1524" layer="91"/>
-<wire x1="152.4" y1="109.22" x2="152.4" y2="116.84" width="0.1524" layer="91"/>
-<pinref part="U1" gate="PORTA_H" pin="PA10"/>
-<wire x1="152.4" y1="116.84" x2="172.72" y2="116.84" width="0.1524" layer="91"/>
-<pinref part="LED1" gate="G$1" pin="A"/>
-<pinref part="JP2" gate="G$1" pin="1"/>
-<wire x1="152.4" y1="109.22" x2="152.4" y2="99.06" width="0.1524" layer="91"/>
-<wire x1="152.4" y1="99.06" x2="160.02" y2="99.06" width="0.1524" layer="91"/>
-<junction x="152.4" y="109.22"/>
-</segment>
-</net>
 <net name="N$62" class="0">
 <segment>
@@
 <pinref part="U1" gate="PORTA_H" pin="PA9"/>
 <wire x1="172.72" y1="114.3" x2="213.36" y2="114.3" width="0.1524" layer="91"/>
-<wire x1="213.36" y1="114.3" x2="213.36" y2="149.86" width="0.1524" layer="91"/>
+<wire x1="213.36" y1="114.3" x2="213.36" y2="121.92" width="0.1524" layer="91"/>
 <pinref part="JP4" gate="A" pin="2"/>
+<wire x1="213.36" y1="121.92" x2="213.36" y2="149.86" width="0.1524" layer="91"/>
 <wire x1="213.36" y1="149.86" x2="205.74" y2="149.86" width="0.1524" layer="91"/>
+<pinref part="R1" gate="G$1" pin="1"/>
+<wire x1="238.76" y1="121.92" x2="213.36" y2="121.92" width="0.1524" layer="91"/>
+<junction x="213.36" y="121.92"/>
 </segment>
 </net>
@@
 </segment>
 </net>
+<net name="N$19" class="0">
+<segment>
+<pinref part="U$1" gate="G$1" pin="REFRESH"/>
+<pinref part="U$4" gate="G$1" pin="REFRESH"/>
+<wire x1="449.58" y1="27.94" x2="322.58" y2="27.94" width="0.1524" layer="91"/>
+<pinref part="U$2" gate="G$1" pin="REFRESH"/>
+<wire x1="502.92" y1="27.94" x2="449.58" y2="27.94" width="0.1524" layer="91"/>
+<junction x="449.58" y="27.94"/>
+<pinref part="U$5" gate="G$1" pin="REFRESH"/>
+<wire x1="566.42" y1="27.94" x2="502.92" y2="27.94" width="0.1524" layer="91"/>
+<junction x="502.92" y="27.94"/>
+<pinref part="U$6" gate="G$1" pin="REFRESH"/>
+<wire x1="622.3" y1="27.94" x2="566.42" y2="27.94" width="0.1524" layer="91"/>
+<junction x="566.42" y="27.94"/>
+<pinref part="JP3" gate="-1" pin="REFRESH"/>
+<wire x1="622.3" y1="27.94" x2="647.7" y2="33.02" width="0.1524" layer="91"/>
+<junction x="622.3" y="27.94"/>
+</segment>
+</net>
 <net name="N$12" class="0">
 <segment>
+<pinref part="R1" gate="G$1" pin="2"/>
 <pinref part="LED1" gate="G$1" pin="C"/>
-<pinref part="R1" gate="G$1" pin="2"/>
-</segment>
-</net>
-<net name="N$15" class="0">
-<segment>
+</segment>
+</net>
+<net name="N$21" class="0">
+<segment>
+<pinref part="U1" gate="PORTC_H" pin="PC9"/>
+<wire x1="431.8" y1="-7.62" x2="383.54" y2="-7.62" width="0.1524" layer="91"/>
+<pinref part="U$4" gate="G$1" pin="HALT"/>
+<pinref part="U$1" gate="G$1" pin="HALT"/>
+<wire x1="322.58" y1="30.48" x2="383.54" y2="30.48" width="0.1524" layer="91"/>
+<pinref part="U$2" gate="G$1" pin="HALT"/>
+<wire x1="383.54" y1="30.48" x2="449.58" y2="30.48" width="0.1524" layer="91"/>
+<wire x1="449.58" y1="30.48" x2="502.92" y2="30.48" width="0.1524" layer="91"/>
+<junction x="449.58" y="30.48"/>
+<pinref part="U$5" gate="G$1" pin="HALT"/>
+<wire x1="502.92" y1="30.48" x2="566.42" y2="30.48" width="0.1524" layer="91"/>
+<junction x="502.92" y="30.48"/>
+<pinref part="U$6" gate="G$1" pin="HALT"/>
+<wire x1="566.42" y1="30.48" x2="622.3" y2="30.48" width="0.1524" layer="91"/>
+<junction x="566.42" y="30.48"/>
+<pinref part="JP3" gate="-1" pin="HALT"/>
+<wire x1="622.3" y1="30.48" x2="647.7" y2="35.56" width="0.1524" layer="91"/>
+<junction x="622.3" y="30.48"/>
+<wire x1="383.54" y1="-7.62" x2="383.54" y2="30.48" width="0.1524" layer="91"/>
+<junction x="383.54" y="30.48"/>
+</segment>
+</net>
+<net name="N$27" class="0">
+<segment>
+<wire x1="269.24" y1="116.84" x2="269.24" y2="33.02" width="0.1524" layer="91"/>
+<pinref part="U1" gate="PORTA_H" pin="PA10"/>
+<wire x1="172.72" y1="116.84" x2="269.24" y2="116.84" width="0.1524" layer="91"/>
 <pinref part="U$4" gate="G$1" pin="WAIT"/>
 <pinref part="U$1" gate="G$1" pin="WAIT"/>
+<pinref part="U$2" gate="G$1" pin="WAIT"/>
 <wire x1="322.58" y1="33.02" x2="449.58" y2="33.02" width="0.1524" layer="91"/>
-<pinref part="U$2" gate="G$1" pin="WAIT"/>
 <wire x1="449.58" y1="33.02" x2="502.92" y2="33.02" width="0.1524" layer="91"/>
 <junction x="449.58" y="33.02"/>
@@
 <wire x1="647.7" y1="38.1" x2="622.3" y2="33.02" width="0.1524" layer="91"/>
 <junction x="622.3" y="33.02"/>
-</segment>
-</net>
+<wire x1="269.24" y1="33.02" x2="322.58" y2="33.02" width="0.1524" layer="91"/>
+<junction x="322.58" y="33.02"/>
+</segment>
+</net>

Commit message: board cleanup
Parts:
- removed C11: 100uF, adafruit:C-USC1210
- removed C12: 100nF, SparkFun-Capacitors:CAP0805
Connections:
- net +3V3: no longer C11.1, C12.1
- net GND: no longer C11.2, C12.2
Changed lines of the file:
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@@
 <part name="P+6" library="supply1" deviceset="+5V" device=""/>
 <part name="C10" library="adafruit" deviceset="C-US" device="C1210" value="100uF"/>
-<part name="C11" library="adafruit" deviceset="C-US" device="C1210" value="100uF"/>
-<part name="GND12" library="supply1" deviceset="GND" device=""/>
-<part name="+3V10" library="supply1" deviceset="+3V3" device=""/>
 <part name="GND13" library="supply1" deviceset="GND" device=""/>
 <part name="JP1" library="pinhead" deviceset="PINHD-1X4" device=""/>
@@
 <part name="GND17" library="supply1" deviceset="GND" device=""/>
 <part name="GND18" library="supply1" deviceset="GND" device=""/>
-<part name="C12" library="SparkFun-Capacitors" deviceset="CAP" device="0805" value="100nF"/>
-<part name="GND22" library="supply1" deviceset="GND" device=""/>
-<part name="+3V8" library="supply1" deviceset="+3V3" device=""/>
 <part name="U$4" library="fap_bus_backplane" deviceset="FAP_BUS" device=""/>
 <part name="U$1" library="fap_bus_backplane" deviceset="FAP_BUS" device=""/>
@@
 <instance part="P+6" gate="1" x="322.58" y="152.4" rot="MR0"/>
 <instance part="C10" gate="G$1" x="129.54" y="114.3"/>
-<instance part="C11" gate="G$1" x="-43.18" y="66.04"/>
-<instance part="GND12" gate="1" x="-43.18" y="53.34"/>
-<instance part="+3V10" gate="G$1" x="-43.18" y="76.2"/>
 <instance part="GND13" gate="1" x="129.54" y="106.68"/>
 <instance part="JP1" gate="A" x="454.66" y="17.78" rot="R180"/>
@@
 <instance part="GND17" gate="1" x="464.82" y="-78.74"/>
 <instance part="GND18" gate="1" x="485.14" y="-35.56"/>
-<instance part="C12" gate="G$1" x="2.54" y="63.5" smashed="yes">
-<attribute name="NAME" x="4.064" y="66.421" size="1.778" layer="95"/>
-<attribute name="VALUE" x="-3.556" y="61.341" size="1.778" layer="96"/>
-</instance>
-<instance part="GND22" gate="1" x="2.54" y="50.8"/>
-<instance part="+3V8" gate="G$1" x="2.54" y="76.2"/>
 <instance part="U$4" gate="G$1" x="335.28" y="109.22"/>
 <instance part="U$1" gate="G$1" x="462.28" y="109.22"/>
@@
 </segment>
 <segment>
-<pinref part="C11" gate="G$1" pin="2"/>
-<pinref part="GND12" gate="1" pin="GND"/>
-<wire x1="-43.18" y1="60.96" x2="-43.18" y2="55.88" width="0.1524" layer="91"/>
-</segment>
-<segment>
 <pinref part="C10" gate="G$1" pin="2"/>
 <pinref part="GND13" gate="1" pin="GND"/>
@@
 <pinref part="GND18" gate="1" pin="GND"/>
 <wire x1="485.14" y1="-33.02" x2="474.98" y2="-33.02" width="0.1524" layer="91"/>
-</segment>
-<segment>
-<pinref part="C12" gate="G$1" pin="2"/>
-<wire x1="2.54" y1="60.96" x2="2.54" y2="53.34" width="0.1524" layer="91"/>
-<pinref part="GND22" gate="1" pin="GND"/>
 </segment>
 <segment>
@@
 </segment>
 <segment>
-<pinref part="C11" gate="G$1" pin="1"/>
-<wire x1="-43.18" y1="68.58" x2="-43.18" y2="73.66" width="0.1524" layer="91"/>
-<pinref part="+3V10" gate="G$1" pin="+3V3"/>
-</segment>
-<segment>
-<pinref part="C12" gate="G$1" pin="1"/>
-<wire x1="2.54" y1="68.58" x2="2.54" y2="73.66" width="0.1524" layer="91"/>
-<pinref part="+3V8" gate="G$1" pin="+3V3"/>
-</segment>
-<segment>
