File: FAP_modules/memory_board/memory_board.brd (EAGLE design)
At the start: 100 x 60 mm, 27 parts, among them IC1 74HC32, IC4 74HC245DW, IC5 AT28C256, IC6 74HC00D

Commit message: added all Z80 signals on bus
Parts:
- U$2: value FAP_BUS_FAP_BUS -> FAP_BUS; device cpu_board:FAP_BUS_2X38 -> fap_bus:2X38
Connections:
- net GND: no longer U$2.GND@31, U$2.GND@33
Changed lines of the file:
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@@
 <attribute name="VALUE" x="20.955" y="28.2702" size="1.778" layer="27" ratio="10"/>
 </element>
-<element name="U$2" library="cpu_board" package="FAP_BUS_2X38" value="FAP_BUS_FAP_BUS" x="32.258" y="2.032" smashed="yes"/>
+<element name="U$2" library="fap_bus" package="2X38" value="FAP_BUS" x="32.258" y="2.032" smashed="yes"/>
 <element name="IC4" library="74xx-eu" package="SO20W" value="74HC245DW" x="62.2554" y="14.8844" smashed="yes">
 <attribute name="VALUE" x="58.4454" y="13.1064" size="1.27" layer="27" ratio="10"/>
@@
 <contactref element="U$2" pad="GND@24"/>
 <contactref element="U$2" pad="GND@9"/>
-<contactref element="U$2" pad="GND@33"/>
 <contactref element="U$2" pad="GND@18"/>
 <contactref element="U$2" pad="GND@3"/>
@@
 <contactref element="U$2" pad="GND@37"/>
 <contactref element="U$2" pad="GND@7"/>
-<contactref element="U$2" pad="GND@31"/>
 <contactref element="U$2" pad="GND@27"/>
 <contactref element="U$2" pad="GND@25"/>

Commit message: board cleanup
Other:
- board text added: "FAP80 Memory Board V2 dekuNukem 2016"
- board text removed: "FAP80 Memory Board REV2 dekuNukem 2016"
Changed lines of the file:
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@@
 <wire x1="0" y1="60" x2="0" y2="0" width="0" layer="20"/>
 <text x="20.955" y="48.4632" size="1.778" layer="25">HM62256</text>
-<text x="62.2728" y="52.873" size="1.778" layer="25">FAP80 Memory Board REV2
+<text x="62.2728" y="52.873" size="1.778" layer="25">FAP80 Memory Board V2
 dekuNukem 2016</text>
 <text x="4.5212" y="49.0474" size="1.016" layer="25">  RAM
